File: Hardware/SparkFun_Qwiic_Thermocouple_Amplifier_PCC/SparkFun_Qwiic_Thermocouple_Amplifier_PCC.sch (EAGLE design)
At the start: 26 parts, among them J1 PTH, J2 QWIIC, J3 QWIIC, J5 PCB_THERMOCOUPLE, U1 MCP9600-SMD

Commit message: Design review changes
Parts:
- FD1, FD2, FD3, FD4: value FIDUCIAL1X2 -> FIDUCIALUFIDUCIAL; device SparkFun-Aesthetics:FIDUCIAL1X2 -> SparkFun-Aesthetics:FIDUCIALUFIDUCIAL
- JP1: value JUMPER-SMT_2_NO_SILK -> JUMPER-SMT_2_NC_TRACE_SILK; device SparkFun-Jumpers:JUMPER-SMT_2_NO_SILK -> SparkFun-Jumpers:JUMPER-SMT_2_NC_TRACE_SILK
- LOGO2: value SFE_LOGO_NAME.1_INCH -> SFE_LOGO_NAME_FLAME.1_INCH; device SparkFun-Aesthetics:SFE_LOGO_NAME.1_INCH -> SparkFun-Aesthetics:SFE_LOGO_NAME_FLAME.1_INCH
- R2: value 43k -> (none); device SparkFun-Resistors:43KOHM-0603-1/10W-1% -> SparkFun-Resistors:RESISTORAXIAL-0.3-KIT
Connections:
- net ADDR: now also R2.2; no longer R2.1
- net GND: now also R2.1; no longer R2.2
Other:
- note added: "Clear jumper to disable power LED"
- note added: "MCP9600 Address Selection: 0x60: ADDR tied to GND (defualt) 0x61: R3 = 10k, R2 = 2.2k 0x62: R3 = 10k, R2 = 4.3k 0x63: R3 = 10k, R2 = 7.5k 0x64: R3 = 10k, R2 = 13k 0x65: R3 = 10k, R2 = 22k 0x66: R3 = 10k, R2 = 43k 0x67: ADDR Pin Tied to VDD"
- note removed: "MCP9600 Address Selection: 0x60: ADDR tied to GND 0x61: R3 = 10k, R2 = 2.2k 0x62: R3 = 10k, R2 = 4.3k 0x63: R3 = 10k, R2 = 7.5k 0x64: R3 = 10k, R2 = 13k 0x65: R3 = 10k, R2 = 22k 0x66: R3 = 10k, R2 = 43k (default) 0x67: ADDR Pin Tied to VDD"
- moved on the sheet: C1, R2
Changed lines of the file:
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@@
 <?xml version="1.0" encoding="utf-8"?>
 <!DOCTYPE eagle SYSTEM "eagle.dtd">
-<eagle version="9.4.1">
+<eagle version="9.5.0">
 <drawing>
 <settings>
-<setting alwaysvectorfont="no"/>
+<setting alwaysvectorfont="yes"/>
 <setting verticaltext="up"/>
 </settings>
@@
 <part name="GND5" library="SparkFun" deviceset="GND" device=""/>
 <part name="GND6" library="SparkFun" deviceset="GND" device=""/>
-<part name="JP1" library="SparkFun-Jumpers" deviceset="JUMPER-SMT_2_NO" device="_SILK" package3d_urn="urn:adsk.eagle:package:39279/1" value=""/>
+<part name="JP1" library="SparkFun-Jumpers" deviceset="JUMPER-SMT_2_NC_TRACE" device="_SILK" package3d_urn="urn:adsk.eagle:package:39281/1" value=""/>
 <part name="SUPPLY5" library="SparkFun-PowerSymbols" library_urn="urn:adsk.eagle:library:530" deviceset="3.3V" device=""/>
-<part name="R2" library="SparkFun-Resistors" deviceset="43KOHM" device="-0603-1/10W-1%" value="43k"/>
 <part name="SUPPLY6" library="SparkFun-PowerSymbols" library_urn="urn:adsk.eagle:library:530" deviceset="3.3V" device=""/>
 <part name="GND2" library="SparkFun-PowerSymbols" deviceset="GND" device=""/>
@@
 <part name="J5" library="SparkFun-Electromechanical" deviceset="PCB_THERMOCOUPLE" device=""/>
 <part name="J4" library="SparkFun-Connectors" deviceset="CONN_04" device="1X04_NO_SILK"/>
-<part name="FD1" library="SparkFun-Aesthetics" deviceset="FIDUCIAL" device="1X2"/>
-<part name="FD2" library="SparkFun-Aesthetics" deviceset="FIDUCIAL" device="1X2"/>
-<part name="FD3" library="SparkFun-Aesthetics" deviceset="FIDUCIAL" device="1X2"/>
-<part name="FD4" library="SparkFun-Aesthetics" deviceset="FIDUCIAL" device="1X2"/>
+<part name="FD1" library="SparkFun-Aesthetics" deviceset="FIDUCIAL" device="UFIDUCIAL" value="FIDUCIALUFIDUCIAL"/>
+<part name="FD2" library="SparkFun-Aesthetics" deviceset="FIDUCIAL" device="UFIDUCIAL" value="FIDUCIALUFIDUCIAL"/>
+<part name="FD3" library="SparkFun-Aesthetics" deviceset="FIDUCIAL" device="UFIDUCIAL" value="FIDUCIALUFIDUCIAL"/>
+<part name="FD4" library="SparkFun-Aesthetics" deviceset="FIDUCIAL" device="UFIDUCIAL" value="FIDUCIALUFIDUCIAL"/>
 <part name="JP3" library="SparkFun-Jumpers" deviceset="JUMPER-SMT_2_NC_TRACE" device="_SILK" package3d_urn="urn:adsk.eagle:package:39281/1" value=""/>
-<part name="LOGO2" library="SparkFun-Aesthetics" deviceset="SFE_LOGO_NAME" device=".1_INCH"/>
+<part name="LOGO2" library="SparkFun-Aesthetics" deviceset="SFE_LOGO_NAME_FLAME" device=".1_INCH"/>
 <part name="LOGO3" library="SparkFun-Aesthetics" deviceset="QWIIC_LOGO" device="_5MM"/>
+<part name="R2" library="SparkFun-Resistors" deviceset="RESISTOR" device="AXIAL-0.3-KIT" value=" "/>
 </parts>
 <sheets>
@@
 I2C pullups</text>
 <text x="76.2" y="114.3" size="1.524" layer="97" font="vector">MCP9600 Address Selection:
-0x60: ADDR tied to GND
+0x60: ADDR tied to GND (defualt)
 0x61: R3 = 10k, R2 = 2.2k
 0x62: R3 = 10k, R2 = 4.3k
@@
 0x64: R3 = 10k, R2 = 13k
 0x65: R3 = 10k, R2 = 22k
-0x66: R3 = 10k, R2 = 43k (default)
+0x66: R3 = 10k, R2 = 43k
 0x67: ADDR Pin Tied to VDD </text>
 <text x="239.522" y="7.366" size="2.54" layer="94" font="vector">v10</text>
 <text x="148.844" y="6.858" size="2.54" layer="94" font="vector">Revised by: Alex Wende</text>
+<text x="50.8" y="167.64" size="1.778" layer="97" font="vector">Clear jumper to disable power LED</text>
 </plain>
 <instances>
@@
 <attribute name="VALUE" x="45.72" y="134.366" size="1.778" layer="96" align="top-center"/>
 </instance>
-<instance part="C1" gate="G$1" x="63.5" y="154.94" smashed="yes">
-<attribute name="NAME" x="65.024" y="157.861" size="1.778" layer="95" font="vector"/>
-<attribute name="VALUE" x="65.024" y="152.781" size="1.778" layer="96" font="vector"/>
-</instance>
-<instance part="GND3" gate="1" x="124.46" y="116.84" smashed="yes" rot="MR0">
-<attribute name="VALUE" x="124.46" y="116.586" size="1.778" layer="96" rot="MR0" align="top-center"/>
-</instance>
-<instance part="GND4" gate="1" x="63.5" y="147.32" smashed="yes">
-<attribute name="VALUE" x="63.5" y="147.066" size="1.778" layer="96" align="top-center"/>
+<instance part="C1" gate="G$1" x="101.6" y="152.4" smashed="yes">
+<attribute name="NAME" x="103.124" y="155.321" size="1.778" layer="95" font="vector"/>
+<attribute name="VALUE" x="103.124" y="150.241" size="1.778" layer="96" font="vector"/>
+</instance>
+<instance part="GND3" gate="1" x="127" y="116.84" smashed="yes" rot="MR0">
+<attribute name="VALUE" x="127" y="116.586" size="1.778" layer="96" rot="MR0" align="top-center"/>
+</instance>
+<instance part="GND4" gate="1" x="101.6" y="144.78" smashed="yes">
+<attribute name="VALUE" x="101.6" y="144.526" size="1.778" layer="96" align="top-center"/>
 </instance>
 <instance part="J1" gate="G$1" x="43.18" y="66.04" smashed="yes" rot="MR0">
@@
 <attribute name="VALUE" x="139.7" y="129.54" size="1.778" layer="96" font="vector" rot="MR270" align="top-left"/>
 </instance>
-<instance part="SUPPLY5" gate="G$1" x="63.5" y="162.56" smashed="yes">
-<attribute name="VALUE" x="63.5" y="165.354" size="1.778" layer="96" align="bottom-center"/>
-</instance>
-<instance part="R2" gate="G$1" x="124.46" y="127" smashed="yes" rot="MR270">
-<attribute name="NAME" x="122.936" y="127" size="1.778" layer="95" font="vector" rot="MR270" align="bottom-center"/>
-<attribute name="VALUE" x="125.984" y="127" size="1.778" layer="96" font="vector" rot="MR270" align="top-center"/>
+<instance part="SUPPLY5" gate="G$1" x="101.6" y="160.02" smashed="yes">
+<attribute name="VALUE" x="101.6" y="162.814" size="1.778" layer="96" align="bottom-center"/>
 </instance>
 <instance part="SUPPLY6" gate="G$1" x="175.26" y="147.32" smashed="yes">
@@
 <instance part="JP9" gate="G$1" x="246.38" y="27.94" smashed="yes"/>
 <instance part="JP2" gate="G$1" x="157.48" y="154.94" smashed="yes" rot="MR270">
-<attribute name="NAME" x="155.829" y="157.226" size="1.778" layer="95" font="vector" rot="MR0"/>
 <attribute name="VALUE" x="155.956" y="151.003" size="1.778" layer="96" font="vector" rot="MR180" align="top-left"/>
 </instance>
@@
 <instance part="LOGO2" gate="G$1" x="149.86" y="38.1" smashed="yes"/>
 <instance part="LOGO3" gate="G$1" x="226.06" y="43.18" smashed="yes"/>
+<instance part="R2" gate="G$1" x="127" y="127" smashed="yes" rot="R90">
+<attribute name="NAME" x="125.476" y="127" size="1.778" layer="95" font="vector" rot="R90" align="bottom-center"/>
+<attribute name="VALUE" x="128.524" y="127" size="1.778" layer="96" font="vector" rot="R90" align="top-center"/>
+</instance>
 </instances>
 <busses>
@@
 <pinref part="C1" gate="G$1" pin="2"/>
 <pinref part="GND4" gate="1" pin="GND"/>
-<wire x1="63.5" y1="152.4" x2="63.5" y2="149.86" width="0.1524" layer="91"/>
+<wire x1="101.6" y1="149.86" x2="101.6" y2="147.32" width="0.1524" layer="91"/>
 </segment>
 <segment>
@@
 </segment>
 <segment>
-<pinref part="R2" gate="G$1" pin="2"/>
 <pinref part="GND3" gate="1" pin="GND"/>
-<wire x1="124.46" y1="121.92" x2="124.46" y2="119.38" width="0.1524" layer="91"/>
+<wire x1="127" y1="121.92" x2="127" y2="119.38" width="0.1524" layer="91"/>
+<pinref part="R2" gate="G$1" pin="1"/>
 </segment>
 <segment>
@@
 <pinref part="C1" gate="G$1" pin="1"/>
 <pinref part="SUPPLY5" gate="G$1" pin="3.3V"/>
-<wire x1="63.5" y1="160.02" x2="63.5" y2="162.56" width="0.1524" layer="91"/>
+<wire x1="101.6" y1="157.48" x2="101.6" y2="160.02" width="0.1524" layer="91"/>
 </segment>
 <segment>
@@
 <pinref part="JP1" gate="G$1" pin="1"/>
 <wire x1="137.16" y1="132.08" x2="137.16" y2="134.62" width="0.1524" layer="91"/>
-<pinref part="R2" gate="G$1" pin="1"/>
-<wire x1="137.16" y1="134.62" x2="124.46" y2="134.62" width="0.1524" layer="91"/>
-<wire x1="124.46" y1="134.62" x2="124.46" y2="132.08" width="0.1524" layer="91"/>
+<wire x1="137.16" y1="134.62" x2="127" y2="134.62" width="0.1524" layer="91"/>
+<wire x1="127" y1="134.62" x2="124.46" y2="134.62" width="0.1524" layer="91"/>
+<wire x1="124.46" y1="134.62" x2="127" y2="134.62" width="0.1524" layer="91"/>
+<wire x1="127" y1="134.62" x2="127" y2="132.08" width="0.1524" layer="91"/>
 <wire x1="124.46" y1="134.62" x2="121.92" y2="134.62" width="0.1524" layer="91"/>
 <junction x="124.46" y="134.62"/>
@@
 <wire x1="137.16" y1="134.62" x2="177.8" y2="134.62" width="0.1524" layer="91"/>
 <junction x="137.16" y="134.62"/>
+<pinref part="R2" gate="G$1" pin="2"/>
+<junction x="127" y="134.62"/>
 </segment>
 </net>
